File: Hardware/Top/CouchProtato-TOP.sch (EAGLE design)
At the start: 52 parts, among them SW1 SWITCH.MOM, SW2 SWITCH.MOM, SW5 SWITCH.MOM, U2 NRF52832_MODULE_MDBT42, U4 PCF8523

Commit message: Top schematic finished
Parts:
- removed SW5: SWITCH.MOM, LinnesLab-Switches:SWITCH.MOM
Connections:
- removed net N$16: SW1.1
- removed net N$18: SW1.3, SW1.4
- removed net N$21: SW2.1
- removed net N$22: SW2.3, SW2.4
- removed net N$23: SW5.1
- removed net N$24: SW5.3, SW5.4
- removed net VBATT: U4.VBAT
- new net SW1: SW1.1, SW2.1
- net GND: now also SW1.3, SW1.4, SW2.3, SW2.4, USB2.SHIELD
Other:
- note removed: "Back-up battery if desired"
- moved on the sheet: SW1, SW2

Commit message: Finished routing top and bottom boards
Parts:
- added C22: 100n, LinnesLab-Passives:CAPACITOR0603
- added C23, C24: 47p, LinnesLab-Passives:CAPACITOR0603
- added JP2: (no value), LinnesLab-Switches:JUMPER-SMT_2_NO_SILK
- added LED5: RED, LinnesLab-LED:LED0603
- added LED6: YELLOW, LinnesLab-LED:LED0603
- added R1, R2: 0, LinnesLab-Passives:RESISTOR0603
- added R17, R18: 27, LinnesLab-Passives:RESISTOR0603
- added R19, R20: 1k, LinnesLab-Passives:RESISTOR0603
- added U5: FT231XS, LinnesLab-DigitalIC:FT231XS
Connections:
- removed net BATT: R13.1, R14.2
- removed net CD1: SD2.CARD_DETECT
- removed net CHRG.STAT: CHRG2.STAT, R12.1
- removed net CS.OLED: U3./CS
- removed net DC.OLED: U3.DC/I2C_SA0
- removed net RESET.OLED: U3./RES
- removed net RXD: U2.P0.08
- removed net SD.CS: SD2.CS
- removed net SW1: SW1.1, SW2.1
- removed net TXD: U2.P0.06
- new net !CTS: JP2.2, U5.!CTS
- new net !DTR: U5.!DTR
- new net A4/BATT: R13.1, R14.2, U2.P0.28/AIN4
- new net A6/TIA: U2.P0.30/AIN6
- new net A7/PPG: U2.P0.31/AIN7
- new net D11/SW1: SW1.1, U2.P0.11
- new net D15/SW2: SW2.1, U2.P0.15
- new net D16/CS.OLED: U2.P0.16, U3./CS
- new net D27/CHRG.STATUS: CHRG2.STAT, R12.1, U2.P0.27
- new net D29/LED.CTRL: U2.P0.29/AIN5
- new net D3/RESET.OLED: U2.P0.03/AIN1, U3./RES
- new net D4/DC.OLED: U2.P0.04/AIN2, U3.DC/I2C_SA0
- new net D5/CD1: SD2.CARD_DETECT, U2.P0.05/AIN3
- new net D7/SD.CS: SD2.CS, U2.P0.07
- new net FT3V3: U5.3V3OUT
- new net N$23: R17.2, U5.USBDM
- new net N$24: R18.2, U5.USBDP
- new net N$25: LED5.C, R19.2
- new net N$26: LED6.C, R20.2
- new net RXD.NRF: R1.2, U2.P0.08
- new net RXDFT: R2.1, U5.RXD
- new net RXLED: R19.1, U5.CBUS1
- new net TXD.NRF: R2.2, U2.P0.06
- new net TXDFT: R1.1, U5.TXD
- new net TXLED: R20.1, U5.CBUS2
- net 3.3V: now also C22.2, LED5.A, LED6.A, U5.!RESET, U5.VCCIO
- net GND: now also C22.1, C23.2, C24.1, JP2.1, U5.GND@16, U5.GND@6
- net SCL: now also R9.1; no longer R8.1
- net SDA: now also R8.1; no longer R9.1
- net USB+: now also C23.1, R18.1
- net USB-: now also C24.2, R17.1
- net V_USB: now also U5.VCC
Other:
- note added: "Bridget Eilers Last worked on 6/12/2020"
- note added: "Digital Output"
- note added: "FTDI Serial-to-USB-Converter"
- note added: "I don't remember if CTS needs to be grounded or left floating so here's a jumper to ground so it can be configued either way dynamically."
- note added: "Notes"
- note added: "TXD goes to RX on the other device RXD goes to TX on the other device"
- moved on the sheet: C2, R8, R9, SW1, SW2, U4, XTAL3

Commit message: finished routing bottom board and began top. finished take 003.
Parts:
- added J1: (no value), LinnesLab-Connectors:CONN_07-1.27MM
- renumbered CHRG2 to CHRG, LDO2 to LDO1
Connections:
- net 3.3V: now also J1.4
- net A6/TIA: now also J1.6
- net A7/PPG: now also J1.7
- net D29/LED.CTRL: now also J1.5
- net GND: now also J1.3
- net SCL: now also J1.2
- net SDA: now also J1.1
Other:
- note added: "Connection to bottom board"
Changed lines of the file:
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@@
 <part name="GND2" library="LinnesLab-Symbols" deviceset="GND" device=""/>
 <part name="SD2" library="LinnesLab-Connectors" deviceset="MICROSD" device="" package3d_urn="urn:adsk.eagle:package:17873109/2"/>
-<part name="CHRG2" library="LinnesLab-Power" deviceset="MCP73831" device=""/>
-<part name="LDO2" library="LinnesLab-Power" deviceset="MIC5504" device=""/>
+<part name="CHRG" library="LinnesLab-Power" deviceset="MCP73831" device=""/>
+<part name="LDO1" library="LinnesLab-Power" deviceset="MIC5504" device=""/>
 <part name="D4" library="LinnesLab-DiscreteSemi" deviceset="SCHOTTKY" device="-USC" package3d_urn="urn:adsk.eagle:package:15664784/2"/>
 <part name="D5" library="LinnesLab-DiscreteSemi" deviceset="SCHOTTKY" device="-USC" package3d_urn="urn:adsk.eagle:package:15664784/2"/>
@@
 <part name="SUPPLY1" library="LinnesLab-Symbols" deviceset="3.3V" device=""/>
 <part name="SUPPLY7" library="LinnesLab-Symbols" deviceset="3.3V" device=""/>
+<part name="J1" library="LinnesLab-Connectors" deviceset="CONN_07" device="-1.27MM"/>
+<part name="GND4" library="LinnesLab-Symbols" deviceset="GND" device=""/>
+<part name="SUPPLY8" library="LinnesLab-Symbols" deviceset="3.3V" device=""/>
 </parts>
 <sheets>
@@
 <text x="5.08" y="246.38" size="7.62" layer="97">Bridget Eilers
 Last worked on 6/12/2020</text>
+<text x="165.1" y="238.76" size="1.778" layer="97">Connection to bottom board</text>
 </plain>
 <instances>
@@
 <attribute name="VALUE" x="223.52" y="-31.75" size="1.778" layer="96"/>
 </instance>
-<instance part="CHRG2" gate="G$1" x="111.76" y="-76.2" smashed="yes">
+<instance part="CHRG" gate="G$1" x="111.76" y="-76.2" smashed="yes">
 <attribute name="NAME" x="104.14" y="-70.612" size="1.778" layer="95"/>
 <attribute name="VALUE" x="104.14" y="-83.82" size="1.778" layer="96"/>
 </instance>
-<instance part="LDO2" gate="G$1" x="114.3" y="-45.72" smashed="yes">
+<instance part="LDO1" gate="G$1" x="114.3" y="-45.72" smashed="yes">
 <attribute name="NAME" x="106.68" y="-36.83" size="1.778" layer="95"/>
 <attribute name="VALUE" x="106.68" y="-55.88" size="1.778" layer="96"/>
@@
 <instance part="SUPPLY7" gate="G$1" x="38.1" y="132.08" smashed="yes">
 <attribute name="VALUE" x="38.1" y="134.874" size="1.778" layer="96" align="bottom-center"/>
+</instance>
+<instance part="J1" gate="G$1" x="167.64" y="264.16" smashed="yes">
+<attribute name="VALUE" x="162.56" y="254.254" size="1.778" layer="96" font="vector"/>
+<attribute name="NAME" x="162.56" y="277.368" size="1.778" layer="95" font="vector"/>
+</instance>
+<instance part="GND4" gate="G$1" x="175.26" y="251.46" smashed="yes">
+<attribute name="VALUE" x="175.26" y="251.206" size="1.778" layer="96" align="top-center"/>
+</instance>
+<instance part="SUPPLY8" gate="G$1" x="175.26" y="279.4" smashed="yes">
+<attribute name="VALUE" x="175.26" y="282.194" size="1.778" layer="96" align="bottom-center"/>
 </instance>
 </instances>
@@
 </segment>
 <segment>
-<pinref part="LDO2" gate="G$1" pin="GND"/>
+<pinref part="LDO1" gate="G$1" pin="GND"/>
 <wire x1="104.14" y1="-45.72" x2="99.06" y2="-45.72" width="0.1524" layer="91"/>
 <wire x1="99.06" y1="-45.72" x2="99.06" y2="-58.42" width="0.1524" layer="91"/>
@@
 </segment>
 <segment>
-<pinref part="CHRG2" gate="G$1" pin="VSS"/>
+<pinref part="CHRG" gate="G$1" pin="VSS"/>
 <wire x1="121.92" y1="-78.74" x2="124.46" y2="-78.74" width="0.1524" layer="91"/>
 <pinref part="GND43" gate="G$1" pin="GND"/>
@@
 <pinref part="GND13" gate="G$1" pin="GND"/>
 <pinref part="C2" gate="G$1" pin="2"/>
+</segment>
+<segment>
+<pinref part="J1" gate="G$1" pin="3"/>
+<wire x1="172.72" y1="264.16" x2="175.26" y2="264.16" width="0.1524" layer="91"/>
+<pinref part="GND4" gate="G$1" pin="GND"/>
+<wire x1="175.26" y1="254" x2="175.26" y2="264.16" width="0.1524" layer="91"/>
 </segment>
 </net>
@@
 </segment>
 <segment>
-<pinref part="LDO2" gate="G$1" pin="OUT"/>
+<pinref part="LDO1" gate="G$1" pin="OUT"/>
 <wire x1="121.92" y1="-40.64" x2="127" y2="-40.64" width="0.1524" layer="91"/>
 <pinref part="C6" gate="G$1" pin="1"/>
@@
 <wire x1="38.1" y1="132.08" x2="38.1" y2="129.54" width="0.1524" layer="91"/>
 </segment>
+<segment>
+<pinref part="J1" gate="G$1" pin="4"/>
+<wire x1="172.72" y1="266.7" x2="175.26" y2="266.7" width="0.1524" layer="91"/>
+<pinref part="SUPPLY8" gate="G$1" pin="3.3V"/>
+<wire x1="175.26" y1="279.4" x2="175.26" y2="266.7" width="0.1524" layer="91"/>
+</segment>
 </net>
 <net name="SDA" class="0">
@@
 <label x="27.94" y="116.84" size="1.27" layer="95" rot="R180" xref="yes"/>
 </segment>
+<segment>
+<pinref part="J1" gate="G$1" pin="1"/>
+<wire x1="172.72" y1="259.08" x2="175.26" y2="259.08" width="0.1524" layer="91"/>
+<label x="175.26" y="259.08" size="1.27" layer="95" xref="yes"/>
+</segment>
 </net>
 <net name="SCL" class="0">
@@
 <wire x1="38.1" y1="119.38" x2="38.1" y2="116.84" width="0.1524" layer="91"/>
 <label x="38.1" y="116.84" size="1.27" layer="95" xref="yes"/>
+</segment>
+<segment>
+<pinref part="J1" gate="G$1" pin="2"/>
+<wire x1="172.72" y1="261.62" x2="175.26" y2="261.62" width="0.1524" layer="91"/>
+<label x="175.26" y="261.62" size="1.27" layer="95" xref="yes"/>
 </segment>
 </net>
@@
 <net name="N$17" class="0">
 <segment>
-<pinref part="CHRG2" gate="G$1" pin="PROG"/>
+<pinref part="CHRG" gate="G$1" pin="PROG"/>
 <wire x1="121.92" y1="-76.2" x2="132.08" y2="-76.2" width="0.1524" layer="91"/>
 <pinref part="R11" gate="G$1" pin="2"/>
@@
 </segment>
 <segment>
-<pinref part="CHRG2" gate="G$1" pin="VBAT"/>
+<pinref part="CHRG" gate="G$1" pin="VBAT"/>
 <wire x1="121.92" y1="-73.66" x2="139.7" y2="-73.66" width="0.1524" layer="91"/>
 <pinref part="C20" gate="G$1" pin="1"/>
@@
 <wire x1="71.12" y1="-40.64" x2="78.74" y2="-40.64" width="0.1524" layer="91"/>
 <pinref part="C5" gate="G$1" pin="2"/>
-<pinref part="LDO2" gate="G$1" pin="IN"/>
+<pinref part="LDO1" gate="G$1" pin="IN"/>
 <wire x1="78.74" y1="-40.64" x2="93.98" y2="-40.64" width="0.1524" layer="91"/>
 <wire x1="93.98" y1="-40.64" x2="93.98" y2="-43.18" width="0.1524" layer="91"/>
 <wire x1="104.14" y1="-40.64" x2="101.6" y2="-40.64" width="0.1524" layer="91"/>
 <junction x="93.98" y="-40.64"/>
-<pinref part="LDO2" gate="G$1" pin="EN"/>
+<pinref part="LDO1" gate="G$1" pin="EN"/>
 <wire x1="101.6" y1="-40.64" x2="93.98" y2="-40.64" width="0.1524" layer="91"/>
 <wire x1="104.14" y1="-50.8" x2="101.6" y2="-50.8" width="0.1524" layer="91"/>
@@
 <wire x1="78.74" y1="-73.66" x2="78.74" y2="-40.64" width="0.1524" layer="91"/>
 <junction x="78.74" y="-40.64"/>
-<pinref part="CHRG2" gate="G$1" pin="VIN"/>
+<pinref part="CHRG" gate="G$1" pin="VIN"/>
 <wire x1="101.6" y1="-73.66" x2="93.98" y2="-73.66" width="0.1524" layer="91"/>
 <junction x="78.74" y="-73.66"/>
@@
 <wire x1="93.98" y1="-91.44" x2="99.06" y2="-91.44" width="0.1524" layer="91"/>
 <wire x1="99.06" y1="-91.44" x2="99.06" y2="-78.74" width="0.1524" layer="91"/>
-<pinref part="CHRG2" gate="G$1" pin="STAT"/>
+<pinref part="CHRG" gate="G$1" pin="STAT"/>
 <wire x1="99.06" y1="-78.74" x2="101.6" y2="-78.74" width="0.1524" layer="91"/>
 <label x="99.06" y="-91.44" size="1.27" layer="95" xref="yes"/>
@@
 <label x="73.66" y="88.9" size="1.27" layer="95" rot="R180" xref="yes"/>
 </segment>
+<segment>
+<pinref part="J1" gate="G$1" pin="5"/>
+<wire x1="172.72" y1="269.24" x2="175.26" y2="269.24" width="0.1524" layer="91"/>
+<label x="175.26" y="269.24" size="1.27" layer="95" xref="yes"/>
+</segment>
 </net>
 <net name="A6/TIA" class="0">
@@
 <label x="73.66" y="86.36" size="1.27" layer="95" rot="R180" xref="yes"/>
 </segment>
+<segment>
+<pinref part="J1" gate="G$1" pin="6"/>
+<wire x1="172.72" y1="271.78" x2="175.26" y2="271.78" width="0.1524" layer="91"/>
+<label x="175.26" y="271.78" size="1.27" layer="95" xref="yes"/>
+</segment>
 </net>
 <net name="A7/PPG" class="0">
@@
 <label x="73.66" y="83.82" size="1.27" layer="95" rot="R180" xref="yes"/>
 </segment>
-</net>
+<segment>
+<pinref part="J1" gate="G$1" pin="7"/>
+<wire x1="172.72" y1="274.32" x2="175.26" y2="274.32" width="0.1524" layer="91"/>
+<label x="175.26" y="274.32" size="1.27" layer="95" xref="yes"/>
+</segment>
+</net>

Commit message: Finished take 7, one more how to video to go, reorganizing and finalizing boards
Parts:
- removed C10, C11: 300p, LinnesLab-Passives:CAPACITOR0603
- removed C2: 1u, LinnesLab-Passives:CAPACITOR0603
- removed R15: 100k, LinnesLab-Passives:RESISTOR0603
- removed SD2: (no value), LinnesLab-Connectors:MICROSD
- removed U4: PCF8523, LinnesLab-Clocks:PCF8523
- removed XTAL3: 32.7680kHz, LinnesLab-Clocks:CRYSTALECS-.327-12.5-12-C-TR
- C18: device LinnesLab-Passives:CAPACITOR0402 -> LinnesLab-Passives:CAPACITOR0603
- renumbered C20 to C3, C21 to C4
Connections:
- removed net !DTR: U5.!DTR
- removed net A4/BATT: R13.1, R14.2, U2.P0.28/AIN4
- removed net A6/TIA: J1.6, U2.P0.30/AIN6
- removed net A7/PPG: J1.7, U2.P0.31/AIN7
- removed net CD2: SD2.CARD_DETECT1
- removed net D29/LED.CTRL: J1.5, U2.P0.29/AIN5
- removed net N$19: U4.OSCO, XTAL3.1
- removed net N$20: U4.OSCI, XTAL3.2
- new net A4/PPG: J1.7, U2.P0.28/AIN4
- new net A5/TIA: J1.6, U2.P0.29/AIN5
- new net A7/BATT: R13.1, R14.2, U2.P0.31/AIN7
- new net D30/LED.CTRL: J1.5, U2.P0.30/AIN6
- net 3.3V: no longer C2.1, R15.2, SD2.VDD, U4.VDD
- net D5/CD1: no longer SD2.CARD_DETECT
- net D7/SD.CS: no longer SD2.CS
- net DTR: now also U5.!DTR
- net GND: no longer C10.2, C11.2, C2.2, R15.1, SD2.GND, SD2.GND1, SD2.VSS, U4.VSS
- net MISO: no longer SD2.DATA_OUT
- net MOSI: no longer SD2.DATA_IN
- net P0.09/NFC1: no longer C11.1
- net P0.10/NFC2: no longer C10.1
- net SCK: no longer SD2.SCLK
- net SCL: no longer U4.SCL
- net SDA: no longer U4.SDA
Other:
- note removed: "Connect MISO, MOSI, and SCK to appropriate pins on microcontroller. Those are SPI pins and are generally prespecified. You have more flexibility with the SD.CS pin."
- note removed: "I2C Address = 0x68h"
- note removed: "Real-Time Clock"
- note removed: "SD Card"

Commit message: Finished first revisions of EAGLE designs for smartwatch
Parts:
- removed C19: 2.2uF, LinnesLab-Passives:CAPACITOR0402
- removed C22: 100n, LinnesLab-Passives:CAPACITOR0603
- removed CHRG: MCP73831, LinnesLab-Power:MCP73831
- removed D4: (no value), LinnesLab-DiscreteSemi:SCHOTTKY-USC
- removed LED5: RED, LinnesLab-LED:LED0603
- removed LED6: YELLOW, LinnesLab-LED:LED0603
- removed R18: 27, LinnesLab-Passives:RESISTOR0603
- removed R19: 1k, LinnesLab-Passives:RESISTOR0603
- removed SW2: SWITCH.MOM, LinnesLab-Switches:SWITCH.MOM
- removed U5: FT231XS, LinnesLab-DigitalIC:FT231XS
- added C1: 1u, LinnesLab-Passives:CAPACITOR0603
- added C2: 10u, LinnesLab-Passives:CAPACITOR0805
- added CHRG1: MCP73831, LinnesLab-Power:MCP73831
- added D3: (no value), LinnesLab-DiscreteSemi:SCHOTTKY-USC
- added LED1: RED, LinnesLab-LED:LED0603
- added LED2: BLUE, LinnesLab-LED:LED0603
- added R10: 27, LinnesLab-Passives:RESISTOR0603
- added R16: 0, LinnesLab-Passives:RESISTOR0603
- added RESET: (no value), LinnesLab-Switches:SPST-PTS830GG140-COPY.1-3
- added U1: NRF52832_MODULE_MDBT42, LinnesLab-Microcontrollers:NRF52832_MODULE_MDBT42
- C12: value 10u -> 100n; device LinnesLab-Passives:CAPACITOR0805 -> LinnesLab-Passives:CAPACITOR0603
- C13: value 2.2uF -> 10uF; device LinnesLab-Passives:CAPACITOR0402 -> LinnesLab-Passives:CAPACITOR0603
- C14: value 100n -> 2.2uF; device LinnesLab-Passives:CAPACITOR0603 -> LinnesLab-Passives:CAPACITOR0402
- C15: device LinnesLab-Passives:CAPACITOR0402 -> LinnesLab-Passives:CAPACITOR0603
- C16: value 10uF -> 2.2uF; device LinnesLab-Passives:CAPACITOR0603 -> LinnesLab-Passives:CAPACITOR0402
- C18: device LinnesLab-Passives:CAPACITOR0603 -> LinnesLab-Passives:CAPACITOR0402
- C3: value 4.7u -> (none)
- C6: value 1u -> (none)
- C8: value (none) -> 4.7u
- C9: value (none) -> 100n
- J1: device LinnesLab-Connectors:CONN_07-1.27MM -> LinnesLab-Connectors:CONN_02
- J2: device LinnesLab-Connectors:CONN_02 -> LinnesLab-Connectors:CONN_07-1.27MM
- LED4: value BLUE -> YELLOW
- R1, R2: value 0 -> 10k
- R11: value (none) -> 27
- R12: value 100k -> 10k
- R13: value 100k -> 390k
- R14: value 100k -> 1k
- R17: value 27 -> 0
- R3: value 1k -> 100k
- R4: value 1k -> 5k
- R5, R6: value 10k -> 1k
- R7: value 390k -> 100k
- R8: value 10k -> 100k
- SW1: value SWITCH.MOM -> (none); device LinnesLab-Switches:SWITCH.MOM -> LinnesLab-Switches:SPST-PTS830GG140-COPY.1-3
- SW3, SW4: value (none) -> SWITCH.MOM; device LinnesLab-Switches:SPST-PTS830GG140-COPY.1-3 -> LinnesLab-Switches:SWITCH.MOM
- U2: value NRF52832_MODULE_MDBT42 -> FT231XS; device LinnesLab-Microcontrollers:NRF52832_MODULE_MDBT42 -> LinnesLab-DigitalIC:FT231XS
- renumbered C23 to C11, C24 to C10, CORTEX1 to DEBUG1, D5 to D2, JP2 to JP1, L2 to L1, R20 to R15, USB2 to USB1, XTAL2 to XTAL1
Connections:
- net !CTS: now also U2.!CTS; no longer U5.!CTS
- net 3.3V: now also C18.2, C2.2, C7.1, D3.C, J2.4, LED3.A, LED4.A, R1.2, R2.2, U1.VDD, U2.!RESET, U2.VCCIO; no longer C19.2, C22.2, C6.1, D1.C, J1.4, LED5.A, LED6.A, R5.2, R8.2, U2.VDD, U5.!RESET, U5.VCCIO
- net A4/PPG: now also J2.7, U1.P0.28/AIN4; no longer J1.7, U2.P0.28/AIN4
- net A5/TIA: now also J2.6, U1.P0.29/AIN5; no longer J1.6, U2.P0.29/AIN5
- net A7/BATT: now also R7.1, R8.2, U1.P0.31/AIN7; no longer R13.1, R14.2, U2.P0.31/AIN7
- net D11/SW1: now also SW3.1, U1.P0.11; no longer SW1.1, U2.P0.11
- net D15/SW2: now also SW4.1, U1.P0.15; no longer SW2.1, U2.P0.15
- net D16/CS.OLED: now also U1.P0.16; no longer U2.P0.16
- net D27/CHRG.STATUS: now also CHRG1.STAT, R3.1, U1.P0.27; no longer CHRG.STAT, R12.1, U2.P0.27
- net D3/RESET.OLED: now also U1.P0.03/AIN1; no longer U2.P0.03/AIN1
- net D30/LED.CTRL: now also J2.5, U1.P0.30/AIN6; no longer J1.5, U2.P0.30/AIN6
- net D4/DC.OLED: now also U1.P0.04/AIN2; no longer U2.P0.04/AIN2
- net D5/CD1: now also U1.P0.05/AIN3; no longer U2.P0.05/AIN3
- net D7/SD.CS: now also U1.P0.07; no longer U2.P0.07
- net DFU: now also SW1.B, U1.P0.20; no longer SW3.B, U2.P0.20
- net DTR: now also C9.1, U2.!DTR; no longer C14.1, U5.!DTR
- net FRST: now also U1.P0.22; no longer U2.P0.22
- net FT3V3: now also U2.3V3OUT; no longer U5.3V3OUT
- net GND: now also C1.2, C13.1, C15.1, C2.1, C3.1, C8.2, CHRG1.VSS, J1.1, J2.3, LED1.C, LED2.C, R12.1, R13.2, R4.1, R8.1, RESET.B, SW1.A, SW3.3, SW3.4, SW4.3, SW4.4, U1.GND@1, U1.GND@2, U1.GND@3, U1.GND@4, U2.GND@16, U2.GND@6; no longer C16.1, C19.1, C22.1, C3.2, C8.1, C9.2, CHRG.VSS, J1.3, J2.1, LED3.C, LED4.C, R11.1, R14.1, R6.1, R7.2, SW1.3, SW1.4, SW2.3, SW2.4, SW3.A, SW4.B, U2.GND@1, U2.GND@2, U2.GND@3, U2.GND@4, U5.GND@16, U5.GND@6
- net LED1: now also R5.2, U1.P0.17; no longer R3.2, U2.P0.17
- net LED2: now also R6.2, U1.P0.19; no longer R4.2, U2.P0.19
- net MISO: now also U1.P0.14; no longer U2.P0.14
- net MOSI: now also U1.P0.13; no longer U2.P0.13
- net N$1: now also R12.2; no longer R6.2
- net N$10: now also LED2.A, R6.1; no longer LED4.A, R4.1
- net N$11: now also U1.DCC; no longer U2.DCC
- net N$12: now also C1.1, U1.DEC4; no longer C7.1, U2.DEC4
- net N$13: now also C13.2; no longer C16.2
- net N$15: now also C15.2; no longer C18.2
- net N$16: now also CHRG1.PROG, R4.2; no longer CHRG.PROG, R11.2
- net N$2: now also R13.1; no longer R7.1
- net N$23: now also R10.2, U2.USBDM; no longer R17.2, U5.USBDM
- net N$24: now also R11.2, U2.USBDP; no longer R18.2, U5.USBDP
- net N$25: now also LED3.C, R14.2; no longer LED5.C, R19.2
- net N$26: now also LED4.C; no longer LED6.C
- net N$3: now also C16.2; no longer C13.2
- net N$4: now also C3.2, U1.P0.00/XL1; no longer C8.2, U2.P0.00/XL1
- net N$5: now also C16.1; no longer C13.1
- net N$6: now also C6.1, U1.P0.01/XL2; no longer C9.1, U2.P0.01/XL2
- net N$7: now also C14.2; no longer C15.2
- net N$8: now also C14.1; no longer C15.1
- net N$9: now also LED1.A, R5.1; no longer LED3.A, R3.1
- net P0.09/NFC1: now also U1.P0.09; no longer U2.P0.09
- net P0.10/NFC2: now also U1.P0.10; no longer U2.P0.10
- net RESET: now also C9.2, D3.A, R9.1, RESET.A, U1.P0.21/RESET; no longer C14.2, D1.A, R5.1, SW4.A, U2.P0.21/RESET
- net RXD.NRF: now also R16.2, U1.P0.08; no longer R1.2, U2.P0.08
- net RXDFT: now also R17.1, U2.RXD; no longer R2.1, U5.RXD
- net RXLED: now also R14.1, U2.CBUS1; no longer R19.1, U5.CBUS1
- net SCK: now also U1.P0.12; no longer U2.P0.12
- net SCL: now also J2.2, R2.1, U1.P0.26; no longer J1.2, R9.1, U2.P0.26
- net SDA: now also J2.1, R1.1, U1.P0.25; no longer J1.1, R8.1, U2.P0.25
- net SWCLK: now also U1.SWDCLK; no longer U2.SWDCLK
- net SWDIO: now also U1.SWDIO; no longer U2.SWDIO
- net SWO: now also U1.P0.18/SWO; no longer U2.P0.18/SWO
- net TXD.NRF: now also R17.2, U1.P0.06; no longer R2.2, U2.P0.06
- net TXDFT: now also R16.1, U2.TXD; no longer R1.1, U5.TXD
- net TXLED: now also U2.CBUS2; no longer U5.CBUS2
- net USB+: now also R11.1; no longer R18.1
- net USB-: now also R10.1; no longer R17.1
- net VIN: now also CHRG1.VIN, D1.C, R3.2; no longer CHRG.VIN, D4.C, R12.2
- net VLIPO: now also C8.1, CHRG1.VBAT, D1.A, J1.2, R7.2; no longer C3.1, CHRG.VBAT, D4.A, J2.2, R13.2
- net V_USB: now also U2.VCC; no longer U5.VCC
Other:
- note added: "Bridget Eilers Last worked on 7/1/2020"
- note added: "CouchProtato Top Board"
- note added: "R11 sets charge current I_Charge = 1000/R11"
- note removed: "Bridget Eilers Last worked on 6/12/2020"
- note removed: "Notes"
- moved on the sheet: C12, C13, C14, C15, C16, C17, C18, C3, C4, C5, C6, C7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
