File: Hardware/PPG-Module/CouchProtato-PPG-MODULE.sch (EAGLE design)
At the start: 0 parts

Commit message: Added ppg board and schematic
Parts:
- added LED: (no value), LinnesLab-LED:LED0805
- added PD: (no value), LinnesLab-Sensors:PHOTODIODE2-SMD.GULLWING
- added U$3: (no value), LinnesLab-Connectors:PPG.MODULE.2
Connections:
- new net GND: PD.A, U$3.GND
- new net LED.C: LED.C, U$3.LD1.C
- new net PD.C: PD.C, U$3.PD.C
- new net V+: LED.A, U$3.V+
Other:
- note added: "CouchProtato: PPG Module Revised: 7/6/2020"
